Commit message: working on calibration, corrected sensor mounting position

File: cob_hardware_config/cob3-2b/urdf/calibration_default.urdf.xacro (robot description, xacro)
@@ -50,10 +50,10 @@
 	<property name="def_head_yaw" value="0.0"/>
 	<!-- arm mount positions | relative to base_link -->
-	<property name="def_arm_x" value="0.040"/>
+	<property name="def_arm_x" value="0.020"/> <!-- 0.040 -->
 	<property name="def_arm_y" value="-0.005"/>
-	<property name="def_arm_z" value="0.83637"/>
-	<property name="def_arm_roll" value="3.1415926"/>
-	<property name="def_arm_pitch" value="0.7854"/>
-	<property name="def_arm_yaw" value="-1.8326"/>
+	<property name="def_arm_z" value="0.83637"/>  <!-- 0.83637 -->
+	<property name="def_arm_roll" value="0.1"/>  <!--3.1415926  3. x (new x)-->
+	<property name="def_arm_pitch" value="-0.79"/> <!-- 0.7854  2. y (new y) -->
+	<property name="def_arm_yaw" value="1.0"/> <!-- -1.8326     1. z -->
 	<!-- sdh mount positions | relative to arm_7_link -->
 	<property name="def_sdh_x" value="0.0"/>
@@ -61,6 +61,6 @@
 	<property name="def_sdh_z" value="0.0"/>
 	<property name="def_sdh_roll" value="0.0"/>
-	<property name="def_sdh_pitch" value="3.1415926"/>
-	<property name="def_sdh_yaw" value="0.0"/>
+	<property name="def_sdh_pitch" value="0.0"/> <!--3.1415926-->
+	<property name="def_sdh_yaw" value="0.79"/>
 	<!-- *********************************** -->
 	<!-- kinematic chain reference positions -->
@@ -99,5 +99,5 @@
 	<property name="def_cam_l_roll" value="0.0"/>
 	<property name="def_cam_l_pitch" value="0.0"/>
-	<property name="def_cam_l_yaw" value="3.1415926"/>
+	<property name="def_cam_l_yaw" value="0.0"/>
 	<!-- right | stereo baseline calibration | relative to cam_reference_link -->
 	<property name="def_cam_r_x" value="0.12"/>
@@ -106,5 +106,5 @@
 	<property name="def_cam_r_roll" value="0.0"/>
 	<property name="def_cam_r_pitch" value="0.0"/>
-	<property name="def_cam_r_yaw" value="3.1415926"/>
+	<property name="def_cam_r_yaw" value="0.0"/>
 	<!-- cam3d | handeye calibration | relative to cam_reference_link -->
 	<property name="def_cam3d_x" value="0.06"/>
@@ -113,4 +113,4 @@
 	<property name="def_cam3d_roll" value="0.0"/>
 	<property name="def_cam3d_pitch" value="0.0"/>
-	<property name="def_cam3d_yaw" value="3.1415926"/>
+	<property name="def_cam3d_yaw" value="-3.1415"/>
 </robot>

File: cob_hardware_config/cob3-2b/urdf/cob3-2b.urdf.xacro (robot description, xacro)
@@ -21,5 +21,5 @@
   <include filename="$(find cob_description)/urdf/lookat/lookat.urdf.xacro" />
   <!-- arm -->
-  <include filename="$(find schunk_description)/urdf/lwa/lwa.urdf.xacro" />
+  <include filename="$(find schunk_description)/urdf/lwa4d/lwa4d.urdf.xacro" />
   <!-- sdh -->
   <include filename="$(find schunk_description)/urdf/sdh/sdh.urdf.xacro" />
@@ -34,7 +34,13 @@
     <origin xyz="${torso_x} ${torso_y} ${torso_z}" rpy="${torso_roll} ${torso_pitch} ${torso_yaw}" />
   </xacro:torso>
-  <xacro:schunk_lwa name="arm" parent="base_link">
+  <xacro:schunk_lwa4d name="arm" parent="base_link">
     <origin xyz="${arm_x} ${arm_y} ${arm_z}" rpy="${arm_roll} ${arm_pitch} ${arm_yaw}" />
-  </xacro:schunk_lwa>
+  </xacro:schunk_lwa4d>
+  <joint name="arm_toolchanger_fixed_joint" type="fixed">
+    <parent link="arm_7_link" />
+    <child link = "arm_toolchanger_link" />
+    <origin xyz="0.0 0.0 0.095" rpy="0.0 0.0 0.0" />
+  </joint>
+  <link name="arm_toolchanger_link" />
   <xacro:head name="head" parent="torso_upper_neck_tilt_link">
     <origin xyz="${head_x} ${head_y} ${head_z}" rpy="${head_roll} ${head_pitch} ${head_yaw}" />
@@ -44,5 +50,5 @@
     <axis xyz="-1 0 0"/>
   </xacro:lookat>
-  <xacro:schunk_sdh name="sdh" parent="arm_7_link">
+  <xacro:schunk_sdh name="sdh" parent="arm_toolchanger_link">
     <origin xyz="${sdh_x} ${sdh_y} ${sdh_z}" rpy="${sdh_roll} ${sdh_pitch} ${sdh_yaw}" />
   </xacro:schunk_sdh>
