Commit message: using high res sensorring Asus driver, corrected all Asus mounting positions

File: cob_hardware_config/robots/cob4-10/urdf/calibration_default.urdf.xacro (robot description, xacro)
@@ -84,5 +84,5 @@
 	<xacro:property name="def_torso_cam3d_left_x" value="0.125"/>
 	<xacro:property name="def_torso_cam3d_left_y" value="0.01802"/>
-	<xacro:property name="def_torso_cam3d_left_z" value="0.24214"/>
+	<xacro:property name="def_torso_cam3d_left_z" value="0.31214"/>
 	<xacro:property name="def_torso_cam3d_left_roll" value="1.57079"/>
 	<xacro:property name="def_torso_cam3d_left_pitch" value="0.0"/>
@@ -91,5 +91,5 @@
 	<xacro:property name="def_torso_cam3d_right_x" value="0.12839"/>
 	<xacro:property name="def_torso_cam3d_right_y" value="-0.01802"/>
-	<xacro:property name="def_torso_cam3d_right_z" value="0.24214"/>
+	<xacro:property name="def_torso_cam3d_right_z" value="0.31214"/>
 	<xacro:property name="def_torso_cam3d_right_roll" value="1.57079"/>
 	<xacro:property name="def_torso_cam3d_right_pitch" value="0.0"/>
@@ -110,7 +110,7 @@
 	<xacro:property name="def_sensorring_cam3d_front_yaw" value="0.0"/>
 	<!-- cam3d | handeye calibration | relative to sensorring_link -->
-	<xacro:property name="def_sensorring_cam3d_back_x" value="-0.096"/>
-	<xacro:property name="def_sensorring_cam3d_back_y" value="0.0"/>
-	<xacro:property name="def_sensorring_cam3d_back_z" value="0.0195"/>
+	<xacro:property name="def_sensorring_cam3d_back_x" value="-0.121"/>
+	<xacro:property name="def_sensorring_cam3d_back_y" value="-0.095"/>
+	<xacro:property name="def_sensorring_cam3d_back_z" value="0.0293"/>
 	<xacro:property name="def_sensorring_cam3d_back_roll" value="0.0"/>
 	<xacro:property name="def_sensorring_cam3d_back_pitch" value="0.0"/>

Commit message: ropha bringup rc_visard modification

File: cob_hardware_config/robots/cob4-10/urdf/calibration_default.urdf.xacro (robot description, xacro)
@@ -102,11 +102,18 @@
 	<xacro:property name="def_torso_cam3d_down_pitch" value="0.61086"/>
 	<xacro:property name="def_torso_cam3d_down_yaw" value="0.0"/>
-	<!-- cam3d | handeye calibration | relative to sensorring_link -->
-	<xacro:property name="def_sensorring_cam3d_front_x" value="0.096"/>
+	<!-- cam3d RC Visard 160 | handeye calibration | relative to sensorring_link -->
+	<xacro:property name="def_sensorring_cam3d_front_x" value="0.122"/>
+	<xacro:property name="def_sensorring_cam3d_front_y" value="0.081"/>
+	<xacro:property name="def_sensorring_cam3d_front_z" value="0.040"/>
+	<xacro:property name="def_sensorring_cam3d_front_roll" value="-1.57079"/>
+	<xacro:property name="def_sensorring_cam3d_front_pitch" value="0.0"/>
+	<xacro:property name="def_sensorring_cam3d_front_yaw" value="-1.57079"/>
+	<!-- cam3d SICK Visionary T | handeye calibration | relative to sensorring_link -->
+	<!--xacro:property name="def_sensorring_cam3d_front_x" value="0.096"/>
 	<xacro:property name="def_sensorring_cam3d_front_y" value="0.0"/>
 	<xacro:property name="def_sensorring_cam3d_front_z" value="0.0195"/>
 	<xacro:property name="def_sensorring_cam3d_front_roll" value="3.14"/>
 	<xacro:property name="def_sensorring_cam3d_front_pitch" value="0.38"/>
-	<xacro:property name="def_sensorring_cam3d_front_yaw" value="0.0"/>
+	<xacro:property name="def_sensorring_cam3d_front_yaw" value="0.0"/-->
 	<!-- cam3d | handeye calibration | relative to sensorring_link -->
 	<xacro:property name="def_sensorring_cam3d_back_x" value="-0.096"/>

File: cob_hardware_config/robots/cob4-10/urdf/cob4-10.urdf.xacro (robot description, xacro)
@@ -22,4 +22,5 @@
   <xacro:include filename="$(find cob_description)/urdf/sensors/realsense.urdf.xacro" />
   <xacro:include filename="$(find cob_description)/urdf/sensors/kinect.urdf.xacro" />
+  <xacro:include filename="$(find cob_description)/urdf/sensors/rc_visard160.urdf.xacro" />
   <xacro:include filename="$(find cob_description)/urdf/sensors/usb_cam.urdf.xacro" />
   <xacro:include filename="$(find cob_description)/urdf/sensors/sick_3dcs.urdf.xacro" />
@@ -62,10 +63,13 @@
   </xacro:sensorring>
   <!-- cameras -->
-  <xacro:sick_3dcs name="sensorring_cam3d_front" ros_topic="sensorring_cam3d_front" parent="sensorring_link">
+  <xacro:rc_160 prefix="sensorring_cam3d_front_" parent="sensorring_link">
     <origin xyz="${sensorring_cam3d_front_x} ${sensorring_cam3d_front_y} ${sensorring_cam3d_front_z}" rpy="${sensorring_cam3d_front_roll} ${sensorring_cam3d_front_pitch} ${sensorring_cam3d_front_yaw}" />
-  </xacro:sick_3dcs>
-  <xacro:cob_kinect_v0 name="sensorring_cam3d_back" ros_topic="sensorring_cam3d_back" parent="sensorring_link" update_rate="30" data_skip="9">
+  </xacro:rc_160>
+  <!--xacro:sick_3dcs name="sensorring_cam3d_front" ros_topic="sensorring_cam3d_front" parent="sensorring_link">
+    <origin xyz="${sensorring_cam3d_front_x} ${sensorring_cam3d_front_y} ${sensorring_cam3d_front_z}" rpy="${sensorring_cam3d_front_roll} ${sensorring_cam3d_front_pitch} ${sensorring_cam3d_front_yaw}" />
+  </xacro:sick_3dcs-->
+  <!--xacro:cob_kinect_v0 name="sensorring_cam3d_back" ros_topic="sensorring_cam3d_back" parent="sensorring_link" update_rate="30" data_skip="9">
     <origin xyz="${sensorring_cam3d_back_x} ${sensorring_cam3d_back_y} ${sensorring_cam3d_back_z}" rpy="${sensorring_cam3d_back_roll} ${sensorring_cam3d_back_pitch} ${sensorring_cam3d_back_yaw}" />
-  </xacro:cob_kinect_v0>
+  </xacro:cob_kinect_v0-->
   <xacro:cob4_arm name="arm_right" parent="torso_3_link" has_podest="false">
     <origin xyz="${arm_right_x} ${arm_right_y} ${arm_right_z}" rpy="${arm_right_roll} ${arm_right_pitch} ${arm_right_yaw}" />
