Commit message: added calibration values from arm camera calibration

File: cob_hardware_config/robots/raw3-1/urdf/calibration_default.urdf.xacro (robot description, xacro)
@@ -29,10 +29,24 @@
 	<xacro:property name="def_tower_yaw" value="3.14159265359"/>
 	<!--torso mount positions (torso_0_link) | relative to base_link-->
-	<xacro:property name="def_torso_x" value="0.166"/>
+	<!-- Pre-Calibration values -->
+	<!-- <xacro:property name="def_torso_x" value="0.166"/>
 	<xacro:property name="def_torso_y" value="0.2175"/>
 	<xacro:property name="def_torso_z" value="0.302"/>
 	<xacro:property name="def_torso_roll" value="0.0"/>
 	<xacro:property name="def_torso_pitch" value="0.0"/>
-	<xacro:property name="def_torso_yaw" value="1.57079632679"/>
+	<xacro:property name="def_torso_yaw" value="1.57079632679"/> -->
+	<!-- Calibrated values -->
+	<xacro:property name="def_torso_x" value="0.1494"/>
+	<xacro:property name="def_torso_y" value="0.233741"/>
+	<xacro:property name="def_torso_z" value="0.297897"/>
+	<xacro:property name="def_torso_roll" value="-0.00331616"/>
+	<xacro:property name="def_torso_pitch" value="-0.00269065"/>
+	<xacro:property name="def_torso_yaw" value="1.54326"/>
+	<!-- <xacro:property name="def_torso_x" value="0.15454"/>
+	<xacro:property name="def_torso_y" value="0.224087"/>
+	<xacro:property name="def_torso_z" value="0.298804"/>
+	<xacro:property name="def_torso_roll" value="-0.0144334"/>
+	<xacro:property name="def_torso_pitch" value="0.00357975"/>
+	<xacro:property name="def_torso_yaw" value="1.56128"/> -->
 	<!-- head mount positions | relative to head_cover_link -->
 	<xacro:property name="def_head_x" value="0.0"/>
@@ -43,10 +57,24 @@
 	<xacro:property name="def_head_yaw" value="0.0"/>
 	<!--arm mount positions | relative to base_link-->
-	<xacro:property name="def_arm_x" value="0.324"/>
+	<!-- Pre-Calibration values -->
+	<!-- <xacro:property name="def_arm_x" value="0.324"/>
 	<xacro:property name="def_arm_y" value="-0.191"/>
 	<xacro:property name="def_arm_z" value="0.585"/>
 	<xacro:property name="def_arm_roll" value="0.0"/>
 	<xacro:property name="def_arm_pitch" value="0.0"/>
-	<xacro:property name="def_arm_yaw" value="-2.3562"/>
+	<xacro:property name="def_arm_yaw" value="-2.3562"/> -->
+	<!-- Calibrated values -->
+	<xacro:property name="def_arm_x" value="0.306238"/>
+	<xacro:property name="def_arm_y" value="-0.183789"/>
+	<xacro:property name="def_arm_z" value="0.5793"/>
+	<xacro:property name="def_arm_roll" value="0.000849562"/>
+	<xacro:property name="def_arm_pitch" value="0.0225778"/>
+	<xacro:property name="def_arm_yaw" value="-2.36424"/>
+	<!-- <xacro:property name="def_arm_x" value="0.313998"/>
+	<xacro:property name="def_arm_y" value="-0.183157"/>
+	<xacro:property name="def_arm_z" value="0.566428"/>
+	<xacro:property name="def_arm_roll" value="-0.00611175"/>
+	<xacro:property name="def_arm_pitch" value="0.0158204"/>
+	<xacro:property name="def_arm_yaw" value="-2.36499"/> -->
 	<!-- gripper mount positions | relative to arm_ee_link -->
 	<xacro:property name="def_gripper_x" value="0.0"/>

Commit message: removed torso, calibration

File: cob_hardware_config/robots/raw3-1/urdf/calibration_default.urdf.xacro (robot description, xacro)
@@ -65,10 +65,29 @@
 	<xacro:property name="def_arm_yaw" value="-2.3562"/> -->
 	<!-- Calibrated values -->
-	<xacro:property name="def_arm_x" value="0.306238"/>
+	<!-- arm_base_link mount positions | camera_base_calibration | relative to base_link-->
+	<xacro:property name="def_arm_x" value="0.318929"/>
+	<xacro:property name="def_arm_y" value="-0.188408"/>
+	<xacro:property name="def_arm_z" value="0.573711"/>
+	<xacro:property name="def_arm_roll" value="0.0105389"/>
+	<xacro:property name="def_arm_pitch" value="0.014375"/>
+	<xacro:property name="def_arm_yaw" value="-2.36603"/>
+	<!--property name="def_arm_x" value="0.321514"/>
+	<property name="def_arm_y" value="-0.188723"/>
+	<property name="def_arm_z" value="0.575413"/>
+	<property name="def_arm_roll" value="0.00764841"/>
+	<property name="def_arm_pitch" value="0.0187387"/>
+	<property name="def_arm_yaw" value="-2.36936"/-->
+	<!--xacro:property name="def_arm_x" value="0.292915"/>
+	<xacro:property name="def_arm_y" value="-0.151959"/>
+	<xacro:property name="def_arm_z" value="0.570404"/>
+	<xacro:property name="def_arm_roll" value="0.0100785"/>
+	<xacro:property name="def_arm_pitch" value="0.0230791"/>
+	<xacro:property name="def_arm_yaw" value="-2.36751"/-->
+	<!--xacro:property name="def_arm_x" value="0.306238"/>
 	<xacro:property name="def_arm_y" value="-0.183789"/>
 	<xacro:property name="def_arm_z" value="0.5793"/>
 	<xacro:property name="def_arm_roll" value="0.000849562"/>
 	<xacro:property name="def_arm_pitch" value="0.0225778"/>
-	<xacro:property name="def_arm_yaw" value="-2.36424"/>
+	<xacro:property name="def_arm_yaw" value="-2.36424"/-->
 	<!-- <xacro:property name="def_arm_x" value="0.313998"/>
 	<xacro:property name="def_arm_y" value="-0.183157"/>

File: cob_hardware_config/robots/raw3-1/urdf/raw3-1.urdf.xacro (robot description, xacro)
@@ -11,5 +11,5 @@
   <xacro:include filename="$(find raw_description)/urdf/tower_asymetric/tower.urdf.xacro" />
   <!-- torso -->
-  <xacro:include filename="$(find raw_description)/urdf/torso/torso_v2.urdf.xacro" />
+  <!--xacro:include filename="$(find raw_description)/urdf/torso/torso_v2.urdf.xacro" /-->
   <!-- ur_arm -->
   <xacro:include filename="$(find raw_description)/urdf/ur_arm/ur10_arm.urdf.xacro" />
@@ -33,7 +33,7 @@
     <origin xyz="${tower_x} ${tower_y} ${tower_z}" rpy="${tower_roll} ${tower_pitch} ${tower_yaw}" />
   </xacro:tower_asymetric>
-  <xacro:raw_torso_v2 name="torso" parent="base_link">
+  <!--xacro:raw_torso_v2 name="torso" parent="base_link">
     <origin xyz="${torso_x} ${torso_y} ${torso_z}" rpy="${torso_roll} ${torso_pitch} ${torso_yaw}" />
-  </xacro:raw_torso_v2>
+  </xacro:raw_torso_v2-->
   <xacro:ur10 name="arm" parent="base_link">
     <origin xyz="${arm_x} ${arm_y} ${arm_z}" rpy="${arm_roll} ${arm_pitch} ${arm_yaw}" />
